File: Flexboard.sch (EAGLE design)
At the start: 353 parts, among them U1 MK20DN512VLQ10

Commit message: Fixed offset keys
Offset function row keys were offset one key to the right. They are now
correctly lined up so the breaks between each block of function keys are
at the right location
Parts:
- KEY_30, KEY_31, KEY_33: value CHERRY-MX-LED-NOPIN -> CHERRY-MX-LED; device cherrymx:CHERRY-MX-LED-NOPIN -> cherrymx:CHERRY-MX-LED
- KEY_30_OFFSET, KEY_31_OFFSET, KEY_32_OFFSET, KEY_33_OFFSET: value CHERRY-MX-LED -> CHERRY-MX-LED-NOPIN; device cherrymx:CHERRY-MX-LED -> cherrymx:CHERRY-MX-LED-NOPIN
Changed lines of the file:
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@@
 <part name="KEY_28" library="cherrymx" deviceset="CHERRY-MX-LED" device=""/>
 <part name="KEY_29" library="cherrymx" deviceset="CHERRY-MX-LED" device=""/>
-<part name="KEY_30" library="cherrymx" deviceset="CHERRY-MX-LED-NOPIN" device=""/>
-<part name="KEY_31" library="cherrymx" deviceset="CHERRY-MX-LED-NOPIN" device=""/>
+<part name="KEY_30" library="cherrymx" deviceset="CHERRY-MX-LED" device=""/>
+<part name="KEY_31" library="cherrymx" deviceset="CHERRY-MX-LED" device=""/>
 <part name="KEY_32" library="cherrymx" deviceset="CHERRY-MX-LED-NOPIN" device=""/>
-<part name="KEY_33" library="cherrymx" deviceset="CHERRY-MX-LED-NOPIN" device=""/>
+<part name="KEY_33" library="cherrymx" deviceset="CHERRY-MX-LED" device=""/>
 <part name="KEY_34" library="cherrymx" deviceset="CHERRY-MX-LED-NOPIN" device=""/>
 <part name="KEY_35" library="cherrymx" deviceset="CHERRY-MX-LED" device=""/>
@@
 <part name="SJ_R5_1" library="jumper" library_urn="urn:adsk.eagle:library:252" deviceset="SJ" device="W" package3d_urn="urn:adsk.eagle:package:15507/1"/>
 <part name="SJ_R6_1" library="jumper" library_urn="urn:adsk.eagle:library:252" deviceset="SJ" device="W" package3d_urn="urn:adsk.eagle:package:15507/1"/>
-<part name="KEY_30_OFFSET" library="cherrymx" deviceset="CHERRY-MX-LED" device=""/>
-<part name="KEY_31_OFFSET" library="cherrymx" deviceset="CHERRY-MX-LED" device=""/>
-<part name="KEY_32_OFFSET" library="cherrymx" deviceset="CHERRY-MX-LED" device=""/>
-<part name="KEY_33_OFFSET" library="cherrymx" deviceset="CHERRY-MX-LED" device=""/>
+<part name="KEY_30_OFFSET" library="cherrymx" deviceset="CHERRY-MX-LED-NOPIN" device=""/>
+<part name="KEY_31_OFFSET" library="cherrymx" deviceset="CHERRY-MX-LED-NOPIN" device=""/>
+<part name="KEY_32_OFFSET" library="cherrymx" deviceset="CHERRY-MX-LED-NOPIN" device=""/>
+<part name="KEY_33_OFFSET" library="cherrymx" deviceset="CHERRY-MX-LED-NOPIN" device=""/>
 <part name="SJ_LED_R1_0" library="jumper" library_urn="urn:adsk.eagle:library:252" deviceset="SJ" device="W" package3d_urn="urn:adsk.eagle:package:15507/1"/>
 <part name="SJ_LED_R2_0" library="jumper" library_urn="urn:adsk.eagle:library:252" deviceset="SJ" device="W" package3d_urn="urn:adsk.eagle:package:15507/1"/>

Commit message: Fixed net naming to use one indexing for rows and columns
Also fixed naming so that the row wires routed to MCU have useful names
Parts:
- removed SJ_C2, SJ_LED_C2, SJ_LED_R1_0, SJ_LED_R2_1, SJ_LED_R4_0, SJ_R1_0, SJ_R2_1: (no value), jumper:SJW
- added SJ_C20, SJ_LED_C19, SJ_LED_R3_0, SJ_LED_R7_0, SJ_LED_R7_1, SJ_R7_0, SJ_R7_1: (no value), jumper:SJW
- renumbered SJ_LED_C1 to SJ_LED_C20, SJ__LED_R3_0 to SJ__LED_R4_0
Connections:
- removed net COL_0: KEY_1.SW1, KEY_109.SW1, KEY_129.SW1, KEY_21.SW1, KEY_41.SW1, KEY_64.SW1, KEY_87.SW1
- removed net LED_COL_0: KEY_1.LED-, KEY_109.LED-, KEY_129.LED-, KEY_21.LED-, KEY_41.LED-, KEY_64.LED-, KEY_87.LED-
- removed net LED_ROW_0: KEY_1.LED+, KEY_10.LED+, KEY_11.LED+, KEY_12.LED+, KEY_13.LED+, KEY_14.LED+, KEY_15.LED+, KEY_16.LED+, KEY_17.LED+, KEY_18.LED+, KEY_19.LED+, KEY_2.LED+, KEY_20.LED+, KEY_3.LED+, KEY_4.LED+, KEY_5.LED+, KEY_6.LED+, KEY_7.LED+, KEY_8.LED+, KEY_9.LED+
- removed net N$1: KEY_66.LED+, KEY_67.LED+, KEY_68.LED+, KEY_69.LED+, KEY_70.LED+, KEY_71.LED+, KEY_72.LED+, KEY_73.LED+, KEY_74.LED+, KEY_75.LED+, KEY_76.LED+, KEY_77.LED+, KEY_78.LED+, KEY_79.LED+, KEY_80.LED+, KEY_81.LED+, KEY_82.LED+, SJ_LED_R3_1.2, SJ__LED_R4_0.1
- removed net N$138: D111.A, D112.A, D113.A, D114.A, D115.A, D116.A, D117.A, D118.A, D119.A, D120.A, D121.A, D122.A, D123.A, D124.A, D125.A, SJ_R5_0.1, SJ_R5_1.2
- removed net N$157: D131.A, D132.A, D133.A, D134.A, D135.A, D136.A, D137.A, D138.A, D139.A, D140.A, D141.A, SJ_R6_0.1, SJ_R6_1.2
- removed net N$177: KEY_100.LED+, KEY_101.LED+, KEY_102.LED+, KEY_103.LED+, KEY_104.LED+, KEY_89.LED+, KEY_90.LED+, KEY_91.LED+, KEY_92.LED+, KEY_93.LED+, KEY_94.LED+, KEY_95.LED+, KEY_96.LED+, KEY_97.LED+, KEY_98.LED+, KEY_99.LED+, SJ_LED_R4_0.1, SJ_LED_R4_1.2
- removed net N$181: KEY_111.LED+, KEY_112.LED+, KEY_113.LED+, KEY_114.LED+, KEY_115.LED+, KEY_116.LED+, KEY_117.LED+, KEY_118.LED+, KEY_119.LED+, KEY_120.LED+, KEY_121.LED+, KEY_122.LED+, KEY_123.LED+, KEY_124.LED+, KEY_125.LED+, SJ_LED_R5_0.1, SJ_LED_R5_1.2
- removed net N$184: KEY_131.LED+, KEY_132.LED+, KEY_133.LED+, KEY_134.LED+, KEY_135.LED+, KEY_136.LED+, KEY_137.LED+, KEY_138.LED+, KEY_139.LED+, KEY_140.LED+, KEY_141.LED+, SJ_LED_R6_0.1, SJ_LED_R6_1.2
- removed net N$2: KEY_23.LED+, KEY_24.LED+, KEY_25.LED+, KEY_26.LED+, KEY_27.LED+, KEY_28.LED+, KEY_29.LED+, KEY_30.LED+, KEY_30_OFFSET.LED+, KEY_31.LED+, KEY_31_OFFSET.LED+, KEY_32.LED+, KEY_32_OFFSET.LED+, KEY_33.LED+, KEY_33_OFFSET.LED+, KEY_34.LED+, KEY_35.LED+, KEY_36.LED+, KEY_37.LED+, KEY_38.LED+, KEY_39.LED+, KEY_40.LED+, SJ_LED_R1_0.1
- removed net N$61: KEY_43.LED+, KEY_44.LED+, KEY_45.LED+, KEY_46.LED+, KEY_47.LED+, KEY_48.LED+, KEY_49.LED+, KEY_50.LED+, KEY_51.LED+, KEY_52.LED+, KEY_53.LED+, KEY_54.LED+, KEY_55.LED+, KEY_56.LED+, KEY_57.LED+, KEY_58.LED+, KEY_59.LED+, SJ_LED_R2_0.1, SJ_LED_R2_1.2
- removed net N$63: D43.A, D44.A, D45.A, D46.A, D47.A, D48.A, D49.A, D50.A, D51.A, D52.A, D53.A, D54.A, D55.A, D56.A, D57.A, D58.A, D59.A, SJ_R2_0.1, SJ_R2_1.2
- removed net N$91: D66.A, D67.A, D68.A, D69.A, D70.A, D71.A, D72.A, D73.A, D74.A, D75.A, D76.A, D77.A, D78.A, D79.A, D80.A, D81.A, D82.A, SJ_R3_0.1, SJ_R3_1.2
- removed net N$99: D100.A, D101.A, D102.A, D103.A, D104.A, D89.A, D90.A, D91.A, D92.A, D93.A, D94.A, D95.A, D96.A, D97.A, D98.A, D99.A, SJ_R4_0.1, SJ_R4_1.2
- removed net N67: D23.A, D24.A, D25.A, D26.A, D27.A, D28.A, D29.A, D30.A, D31.A, D32.A, D33.A, D34.A, D35.A, D36.A, D37.A, D38.A, D39.A, D40.A, SJ_R1_0.1
- removed net ROW_0: D1.A, D10.A, D11.A, D12.A, D13.A, D14.A, D15.A, D16.A, D17.A, D18.A, D19.A, D2.A, D20.A, D3.A, D4.A, D5.A, D6.A, D7.A, D8.A, D9.A
- new net COL_24: KEY_108.SW1, KEY_145.SW1, KEY_63.SW1, KEY_86.SW1
- new net LED_COL_24: KEY_108.LED-, KEY_145.LED-, KEY_63.LED-, KEY_86.LED-
- new net LED_ROW_2B: KEY_23.LED+, KEY_24.LED+, KEY_25.LED+, KEY_26.LED+, KEY_27.LED+, KEY_28.LED+, KEY_29.LED+, KEY_30.LED+, KEY_30_OFFSET.LED+, KEY_31.LED+, KEY_31_OFFSET.LED+, KEY_32.LED+, KEY_32_OFFSET.LED+, KEY_33.LED+, KEY_33_OFFSET.LED+, KEY_34.LED+, KEY_35.LED+, KEY_36.LED+, KEY_37.LED+, KEY_38.LED+, KEY_39.LED+, KEY_40.LED+, SJ_LED_R2_0.1
- new net LED_ROW_3B: KEY_43.LED+, KEY_44.LED+, KEY_45.LED+, KEY_46.LED+, KEY_47.LED+, KEY_48.LED+, KEY_49.LED+, KEY_50.LED+, KEY_51.LED+, KEY_52.LED+, KEY_53.LED+, KEY_54.LED+, KEY_55.LED+, KEY_56.LED+, KEY_57.LED+, KEY_58.LED+, KEY_59.LED+, SJ_LED_R3_0.1, SJ_LED_R3_1.2
- new net LED_ROW_4B: KEY_66.LED+, KEY_67.LED+, KEY_68.LED+, KEY_69.LED+, KEY_70.LED+, KEY_71.LED+, KEY_72.LED+, KEY_73.LED+, KEY_74.LED+, KEY_75.LED+, KEY_76.LED+, KEY_77.LED+, KEY_78.LED+, KEY_79.LED+, KEY_80.LED+, KEY_81.LED+, KEY_82.LED+, SJ_LED_R4_1.2, SJ__LED_R4_0.1
- new net LED_ROW_5B: KEY_100.LED+, KEY_101.LED+, KEY_102.LED+, KEY_103.LED+, KEY_104.LED+, KEY_89.LED+, KEY_90.LED+, KEY_91.LED+, KEY_92.LED+, KEY_93.LED+, KEY_94.LED+, KEY_95.LED+, KEY_96.LED+, KEY_97.LED+, KEY_98.LED+, KEY_99.LED+, SJ_LED_R5_0.1, SJ_LED_R5_1.2
- new net LED_ROW_6B: KEY_111.LED+, KEY_112.LED+, KEY_113.LED+, KEY_114.LED+, KEY_115.LED+, KEY_116.LED+, KEY_117.LED+, KEY_118.LED+, KEY_119.LED+, KEY_120.LED+, KEY_121.LED+, KEY_122.LED+, KEY_123.LED+, KEY_124.LED+, KEY_125.LED+, SJ_LED_R6_0.1, SJ_LED_R6_1.2
- new net LED_ROW_7: KEY_129.LED+, KEY_130.LED+, SJ_LED_R7_0.2
- new net LED_ROW_7B: KEY_131.LED+, KEY_132.LED+, KEY_133.LED+, KEY_134.LED+, KEY_135.LED+, KEY_136.LED+, KEY_137.LED+, KEY_138.LED+, KEY_139.LED+, KEY_140.LED+, KEY_141.LED+, SJ_LED_R7_0.1, SJ_LED_R7_1.2
- new net ROW_2B: D23.A, D24.A, D25.A, D26.A, D27.A, D28.A, D29.A, D30.A, D31.A, D32.A, D33.A, D34.A, D35.A, D36.A, D37.A, D38.A, D39.A, D40.A, SJ_R2_0.1
- new net ROW_3B: D43.A, D44.A, D45.A, D46.A, D47.A, D48.A, D49.A, D50.A, D51.A, D52.A, D53.A, D54.A, D55.A, D56.A, D57.A, D58.A, D59.A, SJ_R3_0.1, SJ_R3_1.2
- new net ROW_4B: D66.A, D67.A, D68.A, D69.A, D70.A, D71.A, D72.A, D73.A, D74.A, D75.A, D76.A, D77.A, D78.A, D79.A, D80.A, D81.A, D82.A, SJ_R4_0.1, SJ_R4_1.2
- new net ROW_5B: D100.A, D101.A, D102.A, D103.A, D104.A, D89.A, D90.A, D91.A, D92.A, D93.A, D94.A, D95.A, D96.A, D97.A, D98.A, D99.A, SJ_R5_0.1, SJ_R5_1.2
- new net ROW_6B: D111.A, D112.A, D113.A, D114.A, D115.A, D116.A, D117.A, D118.A, D119.A, D120.A, D121.A, D122.A, D123.A, D124.A, D125.A, SJ_R6_0.1, SJ_R6_1.2
- new net ROW_7: D129.A, D130.A, SJ_R7_0.2
- new net ROW_7B: D131.A, D132.A, D133.A, D134.A, D135.A, D136.A, D137.A, D138.A, D139.A, D140.A, D141.A, SJ_R7_0.1, SJ_R7_1.2
- net COL_1: now also KEY_1.SW1, KEY_109.SW1, KEY_129.SW1, KEY_21.SW1, KEY_41.SW1, KEY_64.SW1, KEY_87.SW1; no longer KEY_110.SW1, KEY_130.SW1, KEY_2.SW1, KEY_22.SW1, KEY_42.SW1, KEY_65.SW1, KEY_88.SW1
- net COL_10: now also KEY_118.SW1, KEY_30.SW1, KEY_30_OFFSET.SW1, KEY_50.SW1, KEY_73.SW1, KEY_96.SW1; no longer KEY_119.SW1, KEY_31.SW1, KEY_31_OFFSET.SW1, KEY_51.SW1, KEY_74.SW1, KEY_97.SW1
- net COL_11: now also KEY_119.SW1, KEY_31.SW1, KEY_31_OFFSET.SW1, KEY_51.SW1, KEY_74.SW1, KEY_97.SW1; no longer KEY_120.SW1, KEY_135.SW1, KEY_32.SW1, KEY_32_OFFSET.SW1, KEY_52.SW1, KEY_75.SW1, KEY_98.SW1
- net COL_12: now also KEY_120.SW1, KEY_135.SW1, KEY_32.SW1, KEY_32_OFFSET.SW1, KEY_52.SW1, KEY_75.SW1, KEY_98.SW1; no longer KEY_121.SW1, KEY_136.SW1, KEY_33.SW1, KEY_33_OFFSET.SW1, KEY_53.SW1, KEY_76.SW1, KEY_99.SW1
- net COL_13: now also KEY_121.SW1, KEY_136.SW1, KEY_33.SW1, KEY_33_OFFSET.SW1, KEY_53.SW1, KEY_76.SW1, KEY_99.SW1; no longer KEY_100.SW1, KEY_137.SW1, KEY_34.SW1, KEY_54.SW1, KEY_77.SW1
- net COL_14: now also KEY_100.SW1, KEY_137.SW1, KEY_34.SW1, KEY_54.SW1, KEY_77.SW1; no longer KEY_35.SW1, KEY_55.SW1, KEY_78.SW1
- net COL_15: now also KEY_35.SW1, KEY_55.SW1, KEY_78.SW1; no longer KEY_36.SW1
- net COL_16: now also KEY_36.SW1; no longer KEY_101.SW1, KEY_122.SW1, KEY_138.SW1, KEY_37.SW1, KEY_56.SW1, KEY_79.SW1
- net COL_17: now also KEY_101.SW1, KEY_122.SW1, KEY_138.SW1, KEY_37.SW1, KEY_56.SW1, KEY_79.SW1; no longer KEY_102.SW1, KEY_123.SW1, KEY_139.SW1, KEY_38.SW1, KEY_57.SW1, KEY_80.SW1
- net COL_18: now also KEY_102.SW1, KEY_123.SW1, KEY_139.SW1, KEY_38.SW1, KEY_57.SW1, KEY_80.SW1; no longer KEY_103.SW1, KEY_124.SW1, KEY_140.SW1, KEY_39.SW1, KEY_58.SW1, KEY_81.SW1
- net COL_19: now also KEY_103.SW1, KEY_124.SW1, KEY_140.SW1, KEY_39.SW1, KEY_58.SW1, KEY_81.SW1; no longer KEY_104.SW1, KEY_125.SW1, KEY_141.SW1, KEY_40.SW1, KEY_59.SW1, KEY_82.SW1
- net COL_2: now also KEY_110.SW1, KEY_130.SW1, KEY_2.SW1, KEY_22.SW1, KEY_42.SW1, KEY_65.SW1, KEY_88.SW1; no longer KEY_111.SW1, KEY_131.SW1, KEY_23.SW1, KEY_43.SW1, KEY_66.SW1, KEY_89.SW1, SJ_C2.1
- net COL_20: now also KEY_104.SW1, KEY_125.SW1, KEY_141.SW1, KEY_40.SW1, KEY_59.SW1, KEY_82.SW1, SJ_C20.1; no longer KEY_105.SW1, KEY_126.SW1, KEY_142.SW1, KEY_60.SW1, KEY_83.SW1
- net COL_21: now also KEY_105.SW1, KEY_126.SW1, KEY_142.SW1, KEY_60.SW1, KEY_83.SW1; no longer KEY_106.SW1, KEY_127.SW1, KEY_143.SW1, KEY_61.SW1, KEY_84.SW1
- net COL_22: now also KEY_106.SW1, KEY_127.SW1, KEY_143.SW1, KEY_61.SW1, KEY_84.SW1; no longer KEY_107.SW1, KEY_128.SW1, KEY_144.SW1, KEY_62.SW1, KEY_85.SW1
- net COL_23: now also KEY_107.SW1, KEY_128.SW1, KEY_144.SW1, KEY_62.SW1, KEY_85.SW1; no longer KEY_108.SW1, KEY_145.SW1, KEY_63.SW1, KEY_86.SW1
- net COL_3: now also KEY_111.SW1, KEY_131.SW1, KEY_23.SW1, KEY_43.SW1, KEY_66.SW1, KEY_89.SW1; no longer KEY_112.SW1, KEY_132.SW1, KEY_24.SW1, KEY_44.SW1, KEY_67.SW1, KEY_90.SW1
- net COL_4: now also KEY_112.SW1, KEY_132.SW1, KEY_24.SW1, KEY_44.SW1, KEY_67.SW1, KEY_90.SW1; no longer KEY_113.SW1, KEY_133.SW1, KEY_25.SW1, KEY_45.SW1, KEY_68.SW1, KEY_91.SW1
- net COL_5: now also KEY_113.SW1, KEY_133.SW1, KEY_25.SW1, KEY_45.SW1, KEY_68.SW1, KEY_91.SW1; no longer KEY_114.SW1, KEY_26.SW1, KEY_46.SW1, KEY_69.SW1, KEY_92.SW1
- net COL_6: now also KEY_114.SW1, KEY_26.SW1, KEY_46.SW1, KEY_69.SW1, KEY_92.SW1; no longer KEY_115.SW1, KEY_27.SW1, KEY_47.SW1, KEY_70.SW1, KEY_93.SW1
- net COL_7: now also KEY_115.SW1, KEY_27.SW1, KEY_47.SW1, KEY_70.SW1, KEY_93.SW1; no longer KEY_116.SW1, KEY_134.SW1, KEY_28.SW1, KEY_48.SW1, KEY_71.SW1, KEY_94.SW1
- net COL_8: now also KEY_116.SW1, KEY_134.SW1, KEY_28.SW1, KEY_48.SW1, KEY_71.SW1, KEY_94.SW1; no longer KEY_117.SW1, KEY_29.SW1, KEY_49.SW1, KEY_72.SW1, KEY_95.SW1
- net COL_9: now also KEY_117.SW1, KEY_29.SW1, KEY_49.SW1, KEY_72.SW1, KEY_95.SW1; no longer KEY_118.SW1, KEY_30.SW1, KEY_30_OFFSET.SW1, KEY_50.SW1, KEY_73.SW1, KEY_96.SW1
- net LED_COL_1: now also KEY_1.LED-, KEY_109.LED-, KEY_129.LED-, KEY_21.LED-, KEY_41.LED-, KEY_64.LED-, KEY_87.LED-; no longer KEY_110.LED-, KEY_130.LED-, KEY_2.LED-, KEY_22.LED-, KEY_42.LED-, KEY_65.LED-, KEY_88.LED-
- net LED_COL_10: now also KEY_118.LED-, KEY_30.LED-, KEY_30_OFFSET.LED-, KEY_50.LED-, KEY_73.LED-, KEY_96.LED-; no longer KEY_119.LED-, KEY_31.LED-, KEY_31_OFFSET.LED-, KEY_51.LED-, KEY_74.LED-, KEY_97.LED-
- net LED_COL_11: now also KEY_119.LED-, KEY_31.LED-, KEY_31_OFFSET.LED-, KEY_51.LED-, KEY_74.LED-, KEY_97.LED-; no longer KEY_120.LED-, KEY_135.LED-, KEY_32.LED-, KEY_32_OFFSET.LED-, KEY_52.LED-, KEY_75.LED-, KEY_98.LED-
- net LED_COL_12: now also KEY_120.LED-, KEY_135.LED-, KEY_32.LED-, KEY_32_OFFSET.LED-, KEY_52.LED-, KEY_75.LED-, KEY_98.LED-; no longer KEY_121.LED-, KEY_136.LED-, KEY_33.LED-, KEY_33_OFFSET.LED-, KEY_53.LED-, KEY_76.LED-, KEY_99.LED-
- net LED_COL_13: now also KEY_121.LED-, KEY_136.LED-, KEY_33.LED-, KEY_33_OFFSET.LED-, KEY_53.LED-, KEY_76.LED-, KEY_99.LED-; no longer KEY_100.LED-, KEY_137.LED-, KEY_34.LED-, KEY_54.LED-, KEY_77.LED-
- net LED_COL_14: now also KEY_100.LED-, KEY_137.LED-, KEY_34.LED-, KEY_54.LED-, KEY_77.LED-; no longer KEY_35.LED-, KEY_55.LED-, KEY_78.LED-
- net LED_COL_15: now also KEY_35.LED-, KEY_55.LED-, KEY_78.LED-; no longer KEY_36.LED-
- net LED_COL_16: now also KEY_36.LED-; no longer KEY_101.LED-, KEY_122.LED-, KEY_138.LED-, KEY_37.LED-, KEY_56.LED-, KEY_79.LED-
- net LED_COL_17: now also KEY_101.LED-, KEY_122.LED-, KEY_138.LED-, KEY_37.LED-, KEY_56.LED-, KEY_79.LED-; no longer KEY_102.LED-, KEY_123.LED-, KEY_139.LED-, KEY_38.LED-, KEY_57.LED-, KEY_80.LED-
- net LED_COL_18: now also KEY_102.LED-, KEY_123.LED-, KEY_139.LED-, KEY_38.LED-, KEY_57.LED-, KEY_80.LED-; no longer KEY_103.LED-, KEY_124.LED-, KEY_140.LED-, KEY_39.LED-, KEY_58.LED-, KEY_81.LED-
- net LED_COL_19: now also KEY_103.LED-, KEY_124.LED-, KEY_140.LED-, KEY_39.LED-, KEY_58.LED-, KEY_81.LED-, SJ_LED_C19.1; no longer KEY_104.LED-, KEY_125.LED-, KEY_141.LED-, KEY_40.LED-, KEY_59.LED-, KEY_82.LED-, SJ_LED_C20.1
- net LED_COL_2: now also KEY_110.LED-, KEY_130.LED-, KEY_2.LED-, KEY_22.LED-, KEY_42.LED-, KEY_65.LED-, KEY_88.LED-; no longer KEY_111.LED-, KEY_131.LED-, KEY_23.LED-, KEY_43.LED-, KEY_66.LED-, KEY_89.LED-, SJ_LED_C2.1
- net LED_COL_20: now also KEY_104.LED-, KEY_125.LED-, KEY_141.LED-, KEY_40.LED-, KEY_59.LED-, KEY_82.LED-, SJ_LED_C20.1; no longer KEY_105.LED-, KEY_126.LED-, KEY_142.LED-, KEY_60.LED-, KEY_83.LED-
- net LED_COL_21: now also KEY_105.LED-, KEY_126.LED-, KEY_142.LED-, KEY_60.LED-, KEY_83.LED-; no longer KEY_106.LED-, KEY_127.LED-, KEY_143.LED-, KEY_61.LED-, KEY_84.LED-
- net LED_COL_22: now also KEY_106.LED-, KEY_127.LED-, KEY_143.LED-, KEY_61.LED-, KEY_84.LED-; no longer KEY_107.LED-, KEY_128.LED-, KEY_144.LED-, KEY_62.LED-, KEY_85.LED-
- net LED_COL_23: now also KEY_107.LED-, KEY_128.LED-, KEY_144.LED-, KEY_62.LED-, KEY_85.LED-; no longer KEY_108.LED-, KEY_145.LED-, KEY_63.LED-, KEY_86.LED-
- net LED_COL_3: now also KEY_111.LED-, KEY_131.LED-, KEY_23.LED-, KEY_43.LED-, KEY_66.LED-, KEY_89.LED-; no longer KEY_112.LED-, KEY_132.LED-, KEY_24.LED-, KEY_44.LED-, KEY_67.LED-, KEY_90.LED-
- net LED_COL_4: now also KEY_112.LED-, KEY_132.LED-, KEY_24.LED-, KEY_44.LED-, KEY_67.LED-, KEY_90.LED-; no longer KEY_113.LED-, KEY_25.LED-, KEY_45.LED-, KEY_68.LED-, KEY_91.LED-
- net LED_COL_5: now also KEY_113.LED-, KEY_25.LED-, KEY_45.LED-, KEY_68.LED-, KEY_91.LED-; no longer KEY_114.LED-, KEY_26.LED-, KEY_46.LED-, KEY_69.LED-, KEY_92.LED-
- net LED_COL_6: now also KEY_114.LED-, KEY_26.LED-, KEY_46.LED-, KEY_69.LED-, KEY_92.LED-; no longer KEY_115.LED-, KEY_27.LED-, KEY_47.LED-, KEY_70.LED-, KEY_93.LED-
- net LED_COL_7: now also KEY_115.LED-, KEY_27.LED-, KEY_47.LED-, KEY_70.LED-, KEY_93.LED-; no longer KEY_116.LED-, KEY_134.LED-, KEY_28.LED-, KEY_48.LED-, KEY_71.LED-, KEY_94.LED-
- net LED_COL_8: now also KEY_116.LED-, KEY_134.LED-, KEY_28.LED-, KEY_48.LED-, KEY_71.LED-, KEY_94.LED-; no longer KEY_117.LED-, KEY_29.LED-, KEY_49.LED-, KEY_72.LED-, KEY_95.LED-
- net LED_COL_9: now also KEY_117.LED-, KEY_29.LED-, KEY_49.LED-, KEY_72.LED-, KEY_95.LED-; no longer KEY_118.LED-, KEY_30.LED-, KEY_30_OFFSET.LED-, KEY_50.LED-, KEY_73.LED-, KEY_96.LED-
- net LED_ROW_1: now also KEY_1.LED+, KEY_10.LED+, KEY_11.LED+, KEY_12.LED+, KEY_13.LED+, KEY_14.LED+, KEY_15.LED+, KEY_16.LED+, KEY_17.LED+, KEY_18.LED+, KEY_19.LED+, KEY_2.LED+, KEY_20.LED+, KEY_3.LED+, KEY_4.LED+, KEY_5.LED+, KEY_6.LED+, KEY_7.LED+, KEY_8.LED+, KEY_9.LED+; no longer KEY_21.LED+, KEY_22.LED+, SJ_LED_R1_0.2
- net LED_ROW_2: now also KEY_21.LED+, KEY_22.LED+; no longer KEY_41.LED+, KEY_42.LED+
- net LED_ROW_3: now also KEY_41.LED+, KEY_42.LED+, SJ_LED_R3_0.2; no longer KEY_64.LED+, KEY_65.LED+, SJ__LED_R4_0.2
- net LED_ROW_4: now also KEY_64.LED+, KEY_65.LED+, SJ__LED_R4_0.2; no longer KEY_87.LED+, KEY_88.LED+, SJ_LED_R4_0.2
- net LED_ROW_5: now also KEY_87.LED+, KEY_88.LED+; no longer KEY_109.LED+, KEY_110.LED+
- net LED_ROW_6: now also KEY_109.LED+, KEY_110.LED+; no longer KEY_129.LED+, KEY_130.LED+
- net N$10: now also SJ_C6.2; no longer SJ_C5.2
- net N$103: now also SJ_R5_1.1; no longer SJ_R4_1.1
- net N$124: now also SJ_R6_1.1; no longer SJ_R5_1.1
- net N$14: now also SJ_C7.2; no longer SJ_C6.2
- net N$151: now also SJ_R7_1.1; no longer SJ_R6_1.1
- net N$16: now also SJ_C8.2; no longer SJ_C7.2
- net N$170: now also SJ_LED_R3_1.1; no longer SJ_LED_R2_1.1
- net N$173: now also SJ_LED_R4_1.1; no longer SJ_LED_R3_1.1
- net N$175: now also SJ_LED_C3.2; no longer SJ_LED_C2.2
- net N$179: now also SJ_LED_R5_1.1; no longer SJ_LED_R4_1.1
- net N$18: now also SJ_C9.2; no longer SJ_C8.2
- net N$182: now also SJ_LED_R6_1.1; no longer SJ_LED_R5_1.1
- net N$185: now also SJ_LED_R7_1.1; no longer SJ_LED_R6_1.1
- net N$186: now also SJ_LED_C4.2; no longer SJ_LED_C3.2
- net N$187: now also SJ_LED_C5.2; no longer SJ_LED_C4.2
- net N$188: now also SJ_LED_C6.2; no longer SJ_LED_C5.2
- net N$189: now also SJ_LED_C7.2; no longer SJ_LED_C6.2
- net N$190: now also SJ_LED_C8.2; no longer SJ_LED_C7.2
- net N$191: now also SJ_LED_C9.2; no longer SJ_LED_C8.2
- net N$192: now also SJ_LED_C10.2; no longer SJ_LED_C9.2
- net N$193: now also SJ_LED_C11.2; no longer SJ_LED_C10.2
- net N$194: now also SJ_LED_C12.2; no longer SJ_LED_C11.2
- net N$195: now also SJ_LED_C13.2; no longer SJ_LED_C12.2
- net N$196: now also SJ_LED_C14.2; no longer SJ_LED_C13.2
- net N$197: now also SJ_LED_C15.2; no longer SJ_LED_C14.2
- net N$198: now also SJ_LED_C16.2; no longer SJ_LED_C15.2
- net N$199: now also SJ_LED_C17.2; no longer SJ_LED_C16.2
- net N$200: now also SJ_LED_C18.2; no longer SJ_LED_C17.2
- net N$201: now also SJ_LED_C19.2; no longer SJ_LED_C18.2
- net N$3: now also SJ_C3.2; no longer SJ_C2.2
- net N$4: now also SJ_C4.2; no longer SJ_C3.2
- net N$46: now also SJ_C10.2; no longer SJ_C9.2
- net N$5: now also SJ_C5.2; no longer SJ_C4.2
- net N$50: now also SJ_C11.2; no longer SJ_C10.2
- net N$52: now also SJ_C12.2; no longer SJ_C11.2
- net N$53: now also SJ_C13.2; no longer SJ_C12.2
- net N$54: now also SJ_C14.2; no longer SJ_C13.2
- net N$55: now also SJ_C15.2; no longer SJ_C14.2
- net N$56: now also SJ_C16.2; no longer SJ_C15.2
- net N$57: now also SJ_C17.2; no longer SJ_C16.2
- net N$58: now also SJ_C18.2; no longer SJ_C17.2
- net N$59: now also SJ_C19.2; no longer SJ_C18.2
- net N$60: now also SJ_C20.2; no longer SJ_C19.2
- net N$65: now also SJ_R3_1.1; no longer SJ_R2_1.1
- net N$79: now also SJ_R4_1.1; no longer SJ_R3_1.1
- net ROW_1: now also D1.A, D10.A, D11.A, D12.A, D13.A, D14.A, D15.A, D16.A, D17.A, D18.A, D19.A, D2.A, D20.A, D3.A, D4.A, D5.A, D6.A, D7.A, D8.A, D9.A; no longer D21.A, D22.A, SJ_R1_0.2
- net ROW_2: now also D21.A, D22.A; no longer D41.A, D42.A
- net ROW_3: now also D41.A, D42.A; no longer D64.A, D65.A
- net ROW_4: now also D64.A, D65.A; no longer D87.A, D88.A
- net ROW_5: now also D87.A, D88.A; no longer D109.A, D110.A
- net ROW_6: now also D109.A, D110.A; no longer D129.A, D130.A
Other:
- moved on the sheet: SJ_C10, SJ_C11, SJ_C12, SJ_C13, SJ_C14, SJ_C15, SJ_C16, SJ_C17, SJ_C18, SJ_C19, SJ_C3, SJ_C4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
